File: eagle/tello-charger/tello-charger.brd (EAGLE design)
At the start: 47.9 x 38.1 mm, 11 parts, among them Q1 INKA114AS1

Commit message: [eagle] Update schematic
Routing:
- net N$9: track 44.5 -> 40.1 mm
- net GND: track 91.3 -> 94.6 mm
